Commit message: Here I have fixed the architecture of the project. Also I have found old mistake with differential drive plugin.
TODO
Navigation stack optimization.

File: porter_robot_model/xacro/gazebo_ref.xacro (robot description, xacro)
@@ -12,21 +12,4 @@
 			<robotNamespace>/porter</robotNamespace>
 		</plugin>
-        <plugin name="differential_drive_controller" filename="libgazebo_ros_diff_drive.so" >
-            <commandTopic>${command_topic_name}</commandTopic>
-            <odometryTopic>${odometry_topic_name}</odometryTopic>
-            <odometryFrame>${odometry_topic_name}</odometryFrame>
-            <robotBaseFrame>${base_name}</robotBaseFrame>
-            <publishWheelTF>true</publishWheelTF>
-            <publishWheelJointState>true</publishWheelJointState>
-            <legacyMode>false</legacyMode>
-            <wheelSeparation>${ac_wh_distance}</wheelSeparation>
-            <wheelDiameter>${ac_wh_radius*2}</wheelDiameter>
-            <wheelAcceleration>${wheel_acceleration_gazebo}</wheelAcceleration>
-            <wheelTorque>${wheel_torque_gazebo}</wheelTorque>
-            <updateRate>${update_rate_gazebo}</updateRate>
-            <leftJoint>${left_wheel_joint_name}</leftJoint>
-            <rightJoint>${right_wheel_joint_name}</rightJoint>
-            <publishTf>true</publishTf>
-        </plugin>
     </gazebo>
 </robot>

File: porter_robot_model/xacro/parameters.xacro (robot description, xacro)
@@ -3,15 +3,7 @@
 	<!-- Constants -->
 	<xacro:property name="M_PI" value="3.1415926535897931" />
-	<!-- Topic names -->
-	<xacro:property name="command_topic_name" value="cmd_vel"/>
-	<xacro:property name="odometry_topic_name" value="odom"/>
 	<!-- Link names -->
 	<xacro:property name="base_name" value="chasiss" />
- 	<!-- Joint_names -->
-  	<xacro:property name="left_wheel_joint_name" value="${base_name}_to_left_actuated_wheel"/>
-  	<xacro:property name="right_wheel_joint_name" value="${base_name}_to_right_actuated_wheel"/>
 	<!-- Gazebo parameters -->
-  	<xacro:property name="wheel_torque_gazebo" value="100"/>
-  	<xacro:property name="wheel_acceleration_gazebo" value="100"/>
   	<xacro:property name="update_rate_gazebo" value="50"/>
 	<!-- Parameters of the chasiss -->
@@ -48,5 +40,5 @@
 	<xacro:property name="lidar_posy" value="0.0" />
 	<xacro:property name="lidar_posz" value="0.00" />
-	<xacro:property name="lidar_topic" value="/os1_cloud_node/points" />
+	<xacro:property name="lidar_topic" value="os1_cloud_node/points" />
 	<xacro:property name="lidar_hz" value="10" />
 	<xacro:property name="lidar_lasers" value="64" />

File: porter_robot_model/xacro/sensors/OS1-64.urdf.xacro (robot description, xacro)
@@ -70,5 +70,6 @@
           </ray>
           <plugin name="gazebo_ros_laser_controller" filename="libgazebo_ros_ouster_laser.so">
-            <topicName>${lidar_topic}</topicName>
+          	<robotNamespace>/porter</robotNamespace>
+            <topicName>/porter/${lidar_topic}</topicName>
             <frameName>os1_lidar</frameName>
             <min_range>${lidar_min_range}</min_range>
@@ -81,8 +82,8 @@
   <gazebo>
     <plugin name="imu_controller" filename="libhector_gazebo_ros_imu.so">
-      <robotNamespace>/</robotNamespace>
+      <robotNamespace>/porter</robotNamespace>
       <updateRate>100.0</updateRate>
       <bodyName>os1_imu</bodyName>
-      <topicName>/os1_cloud_node/imu</topicName>
+      <topicName>/porter/os1_cloud_node/imu</topicName>
       <accelDrift>0.005 0.005 0.005</accelDrift>
       <accelGaussianNoise>0.005 0.005 0.005</accelGaussianNoise>
