Commit message: Rebuilded model, temporary removed basler support

File: porter_robot_model/xacro/model.xacro (robot description, xacro)
@@ -22,8 +22,8 @@
 		<xacro:ch_inertial mass="${base_mass}" length="${base_length}" width="${base_width}" thickness="${base_thickness}"/>
 	</link>
- 	<link name="control_box">
+ 	<link name="support">
 		<visual>
 			<geometry>
-				<box size="${cbox_length} ${cbox_width} ${cbox_height}"/>
+				<box size="${support_length} ${support_width} ${support_height}"/>
 			</geometry>
 			<origin rpy="0 0 0" xyz="0 0 0"/>
@@ -32,13 +32,13 @@
 		<collision>
 			<geometry>
-				<box size="${cbox_length} ${cbox_width} ${cbox_height}"/>
+				<box size="${support_length} ${support_width} ${support_height}"/>
 			</geometry>
 		</collision>
-		<xacro:ch_inertial mass="${cbox_mass}" length="${cbox_length}" width="${cbox_width}" thickness="${cbox_height}"/>
+		<xacro:ch_inertial mass="${support_mass}" length="${support_length}" width="${support_width}" thickness="${support_height}"/>
 	</link>
-	<joint name="${base_name}_to_control_box" type="fixed">
+	<joint name="${base_name}_to_support" type="fixed">
 		<parent link="${base_name}"/>
-		<child link="control_box"/>
-		<origin rpy="0 0 0" xyz="0.0 0.0 ${(cbox_height/2+base_thickness/2)}"/>
+		<child link="support"/>
+		<origin rpy="0 0 0" xyz="0.0 0.0 ${(support_height/2+base_thickness/2)}"/>
 	</joint>
 	<xacro:actuated_wheel prefix="right">

File: porter_robot_model/xacro/parameters.xacro (robot description, xacro)
@@ -8,5 +8,4 @@
 	<!-- Link names -->
 	<xacro:property name="base_name" value="chasiss" />
-	<xacro:property name="base_link" value="${base_name}" />
  	<!-- Joint_names -->
   	<xacro:property name="left_wheel_joint_name" value="${base_name}_to_left_actuated_wheel"/>
@@ -21,9 +20,9 @@
 	<xacro:property name="base_thickness" value="0.045" />
 	<xacro:property name="base_mass" value="15"/>
-	<!-- Parameters of the control box -->
-	<xacro:property name="cbox_length" value="0.7" />
-	<xacro:property name="cbox_width" value="0.7" />
-	<xacro:property name="cbox_height" value="0.5" />
-	<xacro:property name="cbox_mass" value="3"/>
+	<!-- Parameters of the support -->
+	<xacro:property name="support_length" value="0.11" />
+	<xacro:property name="support_width" value="0.11" />
+	<xacro:property name="support_height" value="0.18" />
+	<xacro:property name="support_mass" value="3"/>
 	<!-- Parameters of the actuated wheels -->
 	<xacro:property name="ac_wh_distance" value="0.830" />
@@ -42,10 +41,10 @@
 	<!-- Parameters of the camera -->
 	<xacro:property name="camera_box_size" value="0.05" />
-	<xacro:property name="camera_posx" value="0.325" />
+	<xacro:property name="camera_posx" value="0.0" />
 	<xacro:property name="camera_posy" value="-0.10" />
-	<xacro:property name="camera_posz" value="0.00" />
+	<xacro:property name="camera_posz" value="-0.09" />
 	<!-- Parameters of the lidar -->
-	<xacro:property name="lidar_posx" value="0.325" />
-	<xacro:property name="lidar_posy" value="0.10" />
+	<xacro:property name="lidar_posx" value="0.0" />
+	<xacro:property name="lidar_posy" value="0.0" />
 	<xacro:property name="lidar_posz" value="0.00" />
 	<xacro:property name="lidar_topic" value="/os1_cloud_node/points" />

File: porter_robot_model/xacro/sensors/OS1-64.urdf.xacro (robot description, xacro)
@@ -3,6 +3,6 @@
   <!-- <xacro:macro name="OS1-64" params=" name:=  hz:=10 lasers:=64 samples:=512 min_range:=0.9 max_range:=75.0 noise:=0.008 min_angle:=-${M_PI} max_angle:=${M_PI}"> -->
     <joint name="mount_joint" type="fixed">
-      <origin xyz="${lidar_posx} ${lidar_posy} ${cbox_height/2 + 0.073/2 + lidar_posz}" rpy="0 0 0"/>
-      <parent link="control_box"/>
+      <origin xyz="${lidar_posx} ${lidar_posy} ${support_height/2 + 0.073/2 + lidar_posz}" rpy="0 0 0"/>
+      <parent link="support"/>
       <child link="os1_sensor"/>
     </joint>

File: porter_robot_model/xacro/sensors/camera_main.xacro (robot description, xacro)
@@ -24,6 +24,6 @@
 	<joint name="camera_joint" type="fixed">
 		<axis xyz="0 0 0" />
-		<origin xyz="${camera_posx} ${camera_posy} ${cbox_height/2 + camera_box_size/2 + camera_posz}" rpy="0 0 0"/>
-		<parent link="control_box"/>
+		<origin xyz="${camera_posx} ${camera_posy} ${support_height/2 + camera_box_size/2 + camera_posz}" rpy="0 0 0"/>
+		<parent link="support"/>
 		<child link="camera_main"/>
 	</joint>

Commit message: Separated launch of lidar from control. Addition of ODrive USB, want to check the whether bad usb hub was a source of my problems. Small changes in ODrive UART. Hope it will work well. Also I finally remade xacro model to frontal Lidar Placement TODO: Rewrite ODrive USB node

File: porter_robot_model/xacro/model.xacro (robot description, xacro)
@@ -40,5 +40,5 @@
 		<parent link="${base_name}"/>
 		<child link="support"/>
-		<origin rpy="0 0 0" xyz="0.0 0.0 ${(support_height/2+base_thickness/2)}"/>
+		<origin rpy="0 0 0" xyz="0.28 0.0 ${(support_height/2+base_thickness/2)}"/>
 	</joint>
 	<xacro:actuated_wheel prefix="right">

Commit message: experimentation is in progress

File: porter_robot_model/xacro/model.xacro (robot description, xacro)
@@ -6,4 +6,5 @@
 	<xacro:include filename="$(find porter_robot_model)/xacro/sensors/camera_main.xacro"/>
 	<xacro:include filename="$(find porter_robot_model)/xacro/sensors/OS1-64.urdf.xacro"/>
+	<xacro:include filename="$(find porter_robot_model)/xacro/sensors/rs_camera.xacro"/>
 	<!-- Here actual model begins -->
 	<link name="${base_name}">
@@ -37,8 +38,48 @@
 		<xacro:ch_inertial mass="${support_mass}" length="${support_length}" width="${support_width}" thickness="${support_height}"/>
 	</link>
+	<link name="left_camera_support">
+		<visual>
+			<geometry>
+				<box size="0.03 0.03 0.30"/>
+			</geometry>
+			<origin rpy="0 0 0" xyz="0 0 0"/>
+			<material name="blue"/>
+		</visual>
+		<collision>
+			<geometry>
+				<box size="0.03 0.03 0.30"/>
+			</geometry>
+		</collision>
+		<xacro:ch_inertial mass="0.1" length="0.03" width="0.03" thickness="0.30"/>
+	</link>
+	<link name="right_camera_support">
+		<visual>
+			<geometry>
+				<box size="0.03 0.03 0.30"/>
+			</geometry>
+			<origin rpy="0 0 0" xyz="0 0 0"/>
+			<material name="blue"/>
+		</visual>
+		<collision>
+			<geometry>
+				<box size="0.03 0.03 0.30"/>
+			</geometry>
+		</collision>
+		<xacro:ch_inertial mass="0.1" length="0.03" width="0.03" thickness="0.30"/>
+	</link>
 	<joint name="${base_name}_to_support" type="fixed">
 		<parent link="${base_name}"/>
 		<child link="support"/>
 		<origin rpy="0 0 0" xyz="0.28 0.0 ${(support_height/2+base_thickness/2)}"/>
+	</joint>
+	<joint name="${base_name}_to_left_camera_support" type="fixed">
+		<parent link="${base_name}"/>
+		<child link="left_camera_support"/>
+		<origin rpy="0 0 0" xyz="0.33 0.265 ${(0.3/2+base_thickness/2)}"/>
+	</joint>
+	<joint name="${base_name}_to_right_camera_support" type="fixed">
+		<parent link="${base_name}"/>
+		<child link="right_camera_support"/>
+		<origin rpy="0 0 0" xyz="0.33 -0.265 ${(0.3/2+base_thickness/2)}"/>
 	</joint>
 	<xacro:actuated_wheel prefix="right">

File: porter_robot_model/xacro/parameters.xacro (robot description, xacro)
@@ -8,6 +8,6 @@
   	<xacro:property name="update_rate_gazebo" value="50"/>
 	<!-- Parameters of the chasiss -->
-	<xacro:property name="base_length" value="0.7" />
-	<xacro:property name="base_width" value="0.7" />
+	<xacro:property name="base_length" value="0.76" />
+	<xacro:property name="base_width" value="0.76" />
 	<xacro:property name="base_thickness" value="0.045" />
 	<xacro:property name="base_mass" value="15"/>

File: porter_robot_model/xacro/sensors/OS1-64.urdf.xacro (robot description, xacro)
@@ -2,32 +2,44 @@
 <robot xmlns:xacro="http://www.ros.org/wiki/xacro" name="os1_sensor">
   <!-- <xacro:macro name="OS1-64" params=" name:=  hz:=10 lasers:=64 samples:=512 min_range:=0.9 max_range:=75.0 noise:=0.008 min_angle:=-${M_PI} max_angle:=${M_PI}"> -->
-    <joint name="mount_joint" type="fixed">
-      <origin xyz="${lidar_posx} ${lidar_posy} ${support_height/2 + 0.073/2 + lidar_posz}" rpy="0 0 0"/>
-      <parent link="support"/>
-      <child link="os1_sensor"/>
-    </joint>
-    <link name="os1_sensor">
-      <inertial>
-         <mass value="0.33"/>
-         <origin xyz="0 0 0.0365" rpy="0 0 0" />
-         <inertia ixx="0.000241148" ixy="0" ixz="0"
-          iyy="0.000241148" iyz="0" izz="0.000264"/>
-      </inertial>
-      <collision name="base_collision">
-         <origin xyz="0 0 0.0365" rpy="0 0 0" />
-         <geometry>
- 	        <cylinder radius="0.04" length="0.073"/>
-         </geometry>
-      </collision>
-      <visual name="base_visual">
-         <origin xyz="0 0 0.0" rpy="0 0 1.5707" />
-         <geometry>
-	         <mesh filename="package://porter_robot_model/meshes/os1_64.dae" />
-           <!-- <cylinder length="0.073" radius="0.04" /> -->
-         </geometry>
-      </visual>
-    </link>
-    <link name="os1_imu" />
-    <link name="os1_lidar" />
+	<joint name="mount_joint" type="fixed">
+	  <origin xyz="${lidar_posx} ${lidar_posy} ${support_height/2 + 0.073/2 + lidar_posz}" rpy="0 0 0"/>
+	  <parent link="support"/>
+	  <child link="os1_sensor"/>
+	</joint>
+	<link name="os1_sensor">
+	  <inertial>
+		 <mass value="0.33"/>
+		 <origin xyz="0 0 0.0365" rpy="0 0 0" />
+		 <inertia ixx="0.000241148" ixy="0" ixz="0"
+		  iyy="0.000241148" iyz="0" izz="0.000264"/>
+	  </inertial>
+	  <collision>
+		 <origin xyz="0 0 0.0365" rpy="0 0 0" />
+		 <geometry>
+		    <cylinder radius="0.04" length="0.073"/>
+		 </geometry>
+	  </collision>
+	  <visual>
+		 <origin xyz="0 0 0.0" rpy="0 0 1.5707" />
+		 <geometry>
+		     <mesh filename="package://porter_robot_model/meshes/os1_64.dae" />
+		   <!-- <cylinder length="0.073" radius="0.04" /> -->
+		 </geometry>
+	  </visual>
+	</link>
+	<link name="os1_imu">
+		<collision>
+			<geometry>
+				<box size="0.00 0.00 0.0"/>
+			</geometry>
+		</collision>
+	</link>
+    <link name="os1_lidar">
+		<collision>
+			<geometry>
+				<box size="0.00 0.00 0.0"/>
+			</geometry>
+		</collision>
+	</link>
     <joint name="imu_link_joint" type="fixed">
       <parent link="os1_sensor" />
